File: Schematic/USB_Host_Midi_Adapter/USB_Host_Midi_Adapter.kicad_pcb (KiCad board)
At the start: 2 copper layers, 88.3 x 35.6 mm, 37 parts, among them J1 DIN-5, 180°, J2 USB_A, J3 USB_OTG, J4 ICSP_ATMEL, J5 PROG_JMPR, J6 PWR_IN, SW1 SW_RESET, U1 ATMEGA328P-AU, U2 LD1117S33TR_SOT223, U3 MAX3421E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

Commit message: Board complete, dispatch for manufacture
Parts:
- added D1: LED, LEDs:LED_D5.0mm, F.Cu at (199.9, 76.3)
- added R8: 220, Resistors_SMD:R_0805_HandSoldering, F.Cu at (195.3, 76.3)
- C7, C8: value 18pF -> 20pF
- J1: value DIN-5, 180° -> DIN-5_180degree
- Y1, Y2: footprint Crystals:Crystal_SMD_3215-2pin_3.2x1.5mm -> Crystals:Crystal_SMD_3225-4pin_3.2x2.5mm_HandSoldering
- moved C11 7.50 mm to (161.4, 93.6), turned to 180 degrees
- moved C7 3.22 mm to (189.3, 79.8), turned to 270 degrees
- moved C12 2.40 mm to (152.7, 91.3), turned to 90 degrees
- moved C8 2.23 mm to (197.9, 81.9), turned to 90 degrees
- moved Y1 1.72 mm to (193.6, 81.9), turned to 0 degrees
- moved Y2 1.36 mm to (156.3, 90.8), turned to 90 degrees
Connections:
- J2 pad 5: (no net) -> GND
- Y1 pad 2: Net-(C8-Pad2) -> GND
- Y2 pad 2: Net-(C12-Pad2) -> GND
Routing:
- net +5V: track 126.9 -> 154.2 mm
- net Net-(C12-Pad2): track 4.89 -> 10.5 mm
- net Net-(C8-Pad2): track 5.78 -> 10.2 mm
- net Net-(D1-Pad1): track 0.00 -> 3.24 mm
- net Net-(C11-Pad2): track 5.58 -> 7.91 mm
- net Net-(C7-Pad2): track 4.22 -> 6.54 mm
Other:
- board text added: "+5V"
- board text added: "2018 Aidan Lawrence"
- board text added: "GND"
- board text added: "MIDI Helper"
- board text added: "PWR"
- board text added: "REV. 1"
